File: Power.sch (KiCad schematic (older format))
At the start: 35 parts, among them U1 MC34063AD, U2 LM4871

Commit message: shuffled things around
Parts:
- U2: footprint Package_SO:SOIC-8-1EP_3.9x4.9mm_P1.27mm_EP2.35x2.35mm -> Package_SO:SOIC-8_3.9x4.9mm_P1.27mm
Changed lines of the file:
@@
 F 0 "U9" H 3450 4275 50  0000 C CNN
 F 1 "LM4871" H 3450 4184 50  0000 C CNN
-F 2 "Package_SO:SOIC-8-1EP_3.9x4.9mm_P1.27mm_EP2.35x2.35mm" H 3450 4150 50  0001 C CNN
+F 2 "Package_SO:SOIC-8_3.9x4.9mm_P1.27mm" H 3450 4150 50  0001 C CNN
 F 3 "" H 3450 4150 50  0001 C CNN
 	1    3450 4150

Commit message: NTC circuit and values added
Parts:
- U2: symbol ThommasSTUFF:LM4871-Custom_modules -> buttonbox2-rescue:LM4871-Custom_modules-ThommasSTUFF
Changed lines of the file:
@@
 	4550 3100 4550 3000
 $Comp
-L ThommasSTUFF:LM4871-Custom_modules U?
+L buttonbox2-rescue:LM4871-Custom_modules-ThommasSTUFF U?
 U 1 1 5F3EC6A5
 P 3450 4150
