File: buttonbox2.kicad_pcb (KiCad board)
At the start: 2 copper layers, 125 x 209.8 mm, 205 parts, among them J2 AVR-PDI-6, J3 USB_C_Receptacle_USB2.0, J4 Conn_01x03_Male, J6 Micro_SD_Card, Q1 2N7002, SW1 SW_SP3T, SW10 SW_Push, SW11 SW_Push, SW12 SW_Push, SW13 SW_Push, SW14 SW_Push, SW15 SW_Push, SW16 SW_Push, SW17 SW_Push, SW18 SW_Push, SW19 SW_Push, SW2 SW_SPDT, SW20 SW_Push, SW21 SW_Push, SW22 SW_Push, SW23 SW_Push, SW24 SW_Push, SW25 SW_Push, SW26 SW_Push, SW27 SW_Push, SW28 SW_Push, SW29 SW_Push, SW3 Rotary_Encoder_Switch, SW30 SW_Push, SW31 SW_Push, SW32 SW_Push, SW33 SW_Push, SW34 SW_Push, SW35 SW_Push, SW36 SW_Push, SW37 SW_Push, SW38 SW_Push, SW39 SW_Push, SW4 SW_Push, SW5 SW_Push, SW6 SW_Push, SW7 SW_Push, SW8 SW_Push, SW9 SW_Push, U1 ATxmega256A3-AU, U10 MC34063AD, U11 PT6311, U12 VFD_HNV-12SS62, U2 LM4871, U3 YX5200-24SS, U4 SY6926, U5 DMG3415, U6 AMS1117-3.3, U7 DMG3415, U8 LM4871, U9 LM4871, Y2 Crystal_GND24

Commit message: pretty much routed everything
Parts:
- added C37: 100n, Capacitor_SMD:C_0805_2012Metric, B.Cu at (84.1, 30.1)
- added C38: 100n, Capacitor_SMD:C_0805_2012Metric, B.Cu at (93.2, 30.3)
- added C39: 100n, Capacitor_SMD:C_0805_2012Metric, B.Cu at (91.2, 37.7)
- BT1: renamed from BT2; moved to B.Cu
- Cams1, Cbat1, Cbs1, Cbus1, Cin1, Csin1, Csnubber1, Csys1, Ctim1, D6, L1, R28, R35, Rdm1, Rdm2, Rfb1, Ricgh1, Rin1, Risys1, Rnor1, Rsnubber1, TP1, U4, U6, fb2: moved to B.Cu
- moved D4 43.0 mm to (134.0, -47.0)
- moved R34 41.3 mm to (131.2, -24.8), turned to 270 degrees
- moved R26 40.8 mm to (134.0, -43.5), turned to 90 degrees
- moved TP1 37.0 mm to (101.5, -30.2), turned to 180 degrees
- moved R29 32.1 mm to (194.6, -20.8)
- moved SW1 32.1 mm to (197.9, -12.1)
- moved R39 31.9 mm to (123.0, -21.0), turned to 270 degrees
- moved U6 28.1 mm to (100.5, -7.17), turned to 90 degrees
- moved Cbat1 23.0 mm to (101.2, 17.7), turned to 270 degrees
- moved Cin1 21.5 mm to (90.1, -4.22)
- moved BT1 20.0 mm to (98.0, 16.1)
- moved D6 19.8 mm to (110.0, -2.92), turned to 180 degrees
- moved R28 19.8 mm to (106.0, -2.92)
- moved Cams1 17.5 mm to (100.3, -1.68)
- moved Rdm2 14.0 mm to (102.5, 13.0), turned to 270 degrees
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Routing:
- net SYS: track 0.00 -> 355.1 mm, vias 0 -> 12
- net Row6: track 0.00 -> 272.2 mm
- net +3V3: track 0.00 -> 250.9 mm, vias 0 -> 4
- net Row5: track 0.00 -> 242.1 mm, vias 0 -> 8
- net Row4: track 0.00 -> 215.7 mm, vias 0 -> 6
- net Column6: track 0.00 -> 185.2 mm, vias 0 -> 6
- net Row3: track 0.00 -> 178.0 mm, vias 0 -> 4
- net Column1: track 0.00 -> 166.0 mm, vias 0 -> 4
- net Column5: track 0.00 -> 151.1 mm, vias 0 -> 4
- net Column2: track 0.00 -> 150.0 mm, vias 0 -> 4
- net Row2: track 0.00 -> 140.7 mm, vias 0 -> 2
- net Column4: track 0.00 -> 133.1 mm, vias 0 -> 4
- net Column3: track 0.00 -> 133.0 mm, vias 0 -> 4
- net Row1: track 0.00 -> 119.7 mm
- net VEE: track 0.00 -> 111.3 mm, vias 0 -> 2
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- added copper zone on B.Cu, net SIN
- added copper zone on B.Cu, net VIN

Commit message: Fixed some DRC errors and some incorrect wiring
Parts:
- added TH1: Thermistor_NTC, Connector_PinHeader_2.54mm:PinHeader_1x02_P2.54mm_Vertical, F.Cu at (84.1, 19.1)
- moved C35 3.40 mm to (144.3, -3.81), turned to 0 degrees
Connections:
- R34 pad 2: /mainVFD/DOUT -> DOUT
- U1 pad 1: Net-(U1-Pad1) -> Net-(SW1-Pad1)
- U1 pad 20: LED -> STB
- U1 pad 21: Net-(SW1-Pad4) -> DIN
- U1 pad 22: Net-(SW1-Pad2) -> DOUT
- U1 pad 23: Net-(SW1-Pad1) -> CLK
- U1 pad 63: Net-(U1-Pad63) -> Net-(SW1-Pad4)
- U1 pad 64: Net-(U1-Pad64) -> Net-(SW1-Pad2)
- U11 pad 33: Net-(U11-Pad33) -> SYS
- U11 pad 5: /mainVFD/DOUT -> DOUT
- U11 pad 6: Net-(U11-Pad6) -> DIN
- U11 pad 8: Net-(U11-Pad8) -> CLK
- U11 pad 9: Net-(U11-Pad9) -> STB
Routing:
- net DIN: track 0.00 -> 60.0 mm, vias 0 -> 2
- net STB: track 0.00 -> 58.9 mm, vias 0 -> 2
- net DOUT: track 0.00 -> 49.2 mm, vias 0 -> 4
- net CLK: track 0.00 -> 48.6 mm, vias 0 -> 6
- net SYS: track 355.1 -> 374.5 mm, vias 12 -> 14
- net Net-(R35-Pad2): track 0.00 -> 16.2 mm, vias 0 -> 1
- net Net-(SW1-Pad2): track 70.7 -> 82.7 mm, vias 2 -> 6
- net Net-(SW1-Pad1): track 64.8 -> 76.2 mm, vias 2 -> 6
- net Net-(SW1-Pad4): track 66.0 -> 75.3 mm, vias 2 -> 6
- net /mainVFD/DOUT: track 2.68 -> 0.00 mm
- net PGNDBAT: track 28.1 -> 30.0 mm, vias 138 -> 173

Commit message: Added SYS disconnect, routed USB, changed few things
Parts:
- added H1: MountingHole_Pad, MountingHole:MountingHole_2.5mm_Pad, F.Cu at (79.5, -46.6)
- added H2: MountingHole_Pad, MountingHole:MountingHole_2.5mm_Pad, F.Cu at (79.5, 156.4)
- added H3: MountingHole_Pad, MountingHole:MountingHole_2.5mm_Pad, F.Cu at (194.4, -46.6)
- added H4: MountingHole_Pad, MountingHole:MountingHole_2.5mm_Pad, F.Cu at (194.3, 156.4)
- added R40: DNP, Resistor_SMD:R_0805_2012Metric, B.Cu at (101.3, 0.47)
- moved Cams1 1.49 mm to (101.8, -1.68)
- moved Csys1 0.74 mm to (101.3, 2.57)
Connections:
- Cin1 pad 1: VIN -> SIN
- Csys1 pad 1: SYS -> Net-(Csys1-Pad1)
- J3 pad A4: VIN -> SIN
- J3 pad A9: VIN -> SIN
- J3 pad B4: VIN -> SIN
- J3 pad B9: VIN -> SIN
- Rfb1 pad 2: SYS -> Net-(Csys1-Pad1)
- U4 pad 2: VIN -> SIN
- U4 pad 3: SYS -> Net-(Csys1-Pad1)
Routing:
- net D+: track 2.78 -> 104.6 mm, vias 0 -> 2
- net D-: track 2.78 -> 100.9 mm, vias 0 -> 2
- net SIN: track 16.6 -> 48.2 mm, vias 2 -> 6
- net VIN: track 24.4 -> 0.00 mm, vias 2 -> 0
- net SYS: track 374.5 -> 397.9 mm, vias 14 -> 17
- net Net-(Csys1-Pad1): track 0.00 -> 17.3 mm
- net BAT: track 74.2 -> 86.9 mm
- net HW_RX: track 11.6 -> 19.8 mm, vias 0 -> 2
- net Net-(BT1-Pad1): track 36.8 -> 40.2 mm, vias 3 -> 7
- net LX: track 9.45 -> 8.34 mm
- net PGNDBAT: track 30.0 -> 29.4 mm, vias 173 -> 216
- net Net-(R35-Pad2): vias 1 -> 2
- net CLK: vias 6 -> 8
- added copper zone on B.Cu, net LX
Other:
- net class USB added: clearance 0.128, trace_width 0.6, via_dia 0.8, via_drill 0.4
