File: MP3_player.sch (KiCad schematic (older format))
At the start: 32 parts, among them J1 AudioJack3_Ground, J6 Micro_SD_Card, Q1 2N7002, U2 LM4871, U3 YX5200-24SS, U5 DMG3415, U7 DMG3415, U8 LM4871

Commit message: Slight footprint shuffle for the VFD
Parts:
- renumbered LS1 to LSL1, LS2 to LSR1
Changed lines of the file:
@@
 P 9750 4150
 AR Path="/5FDBEEC3" Ref="LS?"  Part="1"
-AR Path="/5FE0503C/5FDBEEC3" Ref="LS1"  Part="1"
+AR Path="/5FE0503C/5FDBEEC3" Ref="LSL1"  Part="1"
 AR Path="/60BB8BC4/5FDBEEC3" Ref="LS?"  Part="1"
-F 0 "LS1" H 9715 3733 50  0000 C CNN
+F 0 "LSL1" H 9715 3733 50  0000 C CNN
 F 1 "Speaker" H 9715 3824 50  0000 C CNN
 F 2 "Connector_Molex:Molex_KK-254_AE-6410-02A_1x02_P2.54mm_Vertical" H 9750 3950 50  0001 C CNN
@@
 P 9850 5600
 AR Path="/618A19C7" Ref="LS?"  Part="1"
-AR Path="/5FE0503C/618A19C7" Ref="LS2"  Part="1"
+AR Path="/5FE0503C/618A19C7" Ref="LSR1"  Part="1"
 AR Path="/60BB8BC4/618A19C7" Ref="LS?"  Part="1"
-F 0 "LS2" H 9815 5183 50  0000 C CNN
+F 0 "LSR1" H 9815 5183 50  0000 C CNN
 F 1 "Speaker" H 9815 5274 50  0000 C CNN
 F 2 "Connector_Molex:Molex_KK-254_AE-6410-02A_1x02_P2.54mm_Vertical" H 9850 5400 50  0001 C CNN

Commit message: Fixed some DRC errors and some incorrect wiring
Parts:
- removed J1: AudioJack3_Ground, symbol Connector:AudioJack3_Ground
Connections:
- no-connect marks 3 -> 11
Changed lines of the file:
@@
 Text HLabel 9100 2200 0    50   Input ~ 0
 SD_CMD
-Text HLabel 9100 2600 0    50   Input ~ 0
-SD_DAT
 Wire Wire Line
 	9150 2600 9100 2600
@@
 Wire Wire Line
 	8350 2350 8350 2400
-Text HLabel 7800 2400 2    50   Input ~ 0
-SD_DAT
 Text HLabel 7800 2500 2    50   Input ~ 0
 SD_CMD
@@
 	1    0    0    -1
 $EndComp
-$Comp
-L Connector:AudioJack3_Ground J1
-U 1 1 60FC2F5F
-P 10600 5000
-F 0 "J1" H 10582 5325 50  0000 C CNN
-F 1 "AudioJack3_Ground" H 10582 5234 50  0000 C CNN
-F 2 "" H 10600 5000 50  0001 C CNN
-F 3 "~" H 10600 5000 50  0001 C CNN
-	1    10600 5000
-	-1   0    0    1
-$EndComp
-$Comp
-L power:GND #PWR052
-U 1 1 60FC4CF9
-P 10700 4550
-AR Path="/5FE0503C/60FC4CF9" Ref="#PWR052"  Part="1"
-AR Path="/60BB8BC4/60FC4CF9" Ref="#PWR?"  Part="1"
-F 0 "#PWR052" H 10700 4300 50  0001 C CNN
-F 1 "GND" H 10705 4377 50  0000 C CNN
-F 2 "" H 10700 4550 50  0001 C CNN
-F 3 "" H 10700 4550 50  0001 C CNN
-	1    10700 4550
-	1    0    0    -1
-$EndComp
-Wire Wire Line
-	10600 4700 10600 4450
-Wire Wire Line
-	10600 4450 10700 4450
-Wire Wire Line
-	10700 4450 10700 4550
+NoConn ~ 9150 2000
+NoConn ~ 9150 2100
+NoConn ~ 9150 2700
+NoConn ~ 7750 2900
+NoConn ~ 7750 3000
+NoConn ~ 6850 2600
+NoConn ~ 6850 2700
+NoConn ~ 6850 2800
+Text HLabel 9100 2600 0    50   Input ~ 0
+SD_DAT
+Text HLabel 7800 2400 2    50   Input ~ 0
+SD_DAT
 $EndSCHEMATC

Commit message: Changed a lot, ordered the final thing
Parts:
- removed Q1: 2N7002, Package_TO_SOT_SMD:SOT-23, symbol Transistor_FET:2N7002
- removed R15: 1K, Resistor_SMD:R_0805_2012Metric, symbol Device:R
- removed R5: 10K, Resistor_SMD:R_0805_2012Metric, symbol Device:R
- removed U5: DMG3415, Package_TO_SOT_SMD:SOT-23, symbol buttonbox2-rescue:DMG3415-custom_comps
- added U5: SN74LV1T34DBV, Package_TO_SOT_SMD:SOT-23-5, symbol Logic_LevelTranslator:SN74LV1T34DBV
- R11, R3: value TBD -> 20K
- R18, R2: value 10K -> 1K
Connections:
- net +5V: now also U5.5 (VCC)
- net AMP_SHDN: now also U5.4 (Y)
- net GND: now also U5.3 (GND)
- net PLAYER_ON: now also U5.2 (A)
- net TX: now also U3.7 (RX)
Other:
- moved on the sheet: R4
Changed lines of the file:
@@
 	1    0    0    -1
 $EndComp
-Text GLabel 6050 2500 0    50   Input ~ 0
+Text GLabel 6850 2500 0    50   Input ~ 0
 TX
-$Comp
-L Device:R R15
-U 1 1 5FE24216
-P 6250 2500
-AR Path="/5FE0503C/5FE24216" Ref="R15"  Part="1"
-AR Path="/60BB8BC4/5FE24216" Ref="R?"  Part="1"
-F 0 "R15" V 6043 2500 50  0000 C CNN
-F 1 "1K" V 6134 2500 50  0000 C CNN
-F 2 "Resistor_SMD:R_0805_2012Metric" V 6180 2500 50  0001 C CNN
-F 3 "~" H 6250 2500 50  0001 C CNN
-	1    6250 2500
-	0    1    1    0
-$EndComp
-Wire Wire Line
-	6850 2500 6400 2500
-Wire Wire Line
-	6100 2500 6050 2500
-Text GLabel 6800 2400 0    50   Input ~ 0
+Text GLabel 6850 2400 0    50   Input ~ 0
 RX
-Wire Wire Line
-	6850 2400 6800 2400
 Wire Wire Line
 	6350 2200 6350 2150
@@
 AR Path="/60BB8BC4/5FE29509" Ref="R?"  Part="1"
 F 0 "R18" V 7343 4150 50  0000 C CNN
-F 1 "10K" V 7434 4150 50  0000 C CNN
+F 1 "1K" V 7434 4150 50  0000 C CNN
 F 2 "Resistor_SMD:R_0805_2012Metric" V 7480 4150 50  0001 C CNN
 F 3 "~" H 7550 4150 50  0001 C CNN
@@
 AR Path="/5FE0503C/5FDBEED0" Ref="U7"  Part="1"
 AR Path="/60BB8BC4/5FDBEED0" Ref="U?"  Part="1"
-F 0 "U7" V 5643 3381 50  0000 C CNN
-F 1 "DMG3415" V 5552 3381 50  0000 C CNN
+F 0 "U7" V 5643 3383 50  0000 C CNN
+F 1 "DMG3415" V 5552 3383 50  0000 C CNN
 F 2 "Package_TO_SOT_SMD:SOT-23" H 5300 3750 50  0001 C CNN
 F 3 "" H 5300 3750 50  0001 C CNN
@@
 	0    1    -1   0
 $EndComp
-Text GLabel 3850 4600 0    50   Input ~ 0
-PLAYER_ON
 Wire Wire Line
 	4750 3650 4600 3650
-$Comp
-L Device:R R?
-U 1 1 5FDBEEE0
-P 4950 4200
-AR Path="/5FDBEEE0" Ref="R?"  Part="1"
-AR Path="/5FE0503C/5FDBEEE0" Ref="R5"  Part="1"
-AR Path="/60BB8BC4/5FDBEEE0" Ref="R?"  Part="1"
-F 0 "R5" H 5020 4246 50  0000 L CNN
-F 1 "10K" H 5020 4155 50  0000 L CNN
-F 2 "Resistor_SMD:R_0805_2012Metric" V 4880 4200 50  0001 C CNN
-F 3 "~" H 4950 4200 50  0001 C CNN
-	1    4950 4200
-	1    0    0    -1
-$EndComp
 $Comp
 L Device:C C?
@@
 	5300 4050 5300 4000
 Wire Wire Line
-	4250 3600 4250 3550
-$Comp
-L Transistor_FET:2N7002 Q?
-U 1 1 5FDBEEF8
-P 4850 4600
-AR Path="/5FDBEEF8" Ref="Q?"  Part="1"
-AR Path="/5FE0503C/5FDBEEF8" Ref="Q1"  Part="1"
-AR Path="/60BB8BC4/5FDBEEF8" Ref="Q?"  Part="1"
-F 0 "Q1" H 5055 4646 50  0000 L CNN
-F 1 "2N7002" H 5055 4555 50  0000 L CNN
-F 2 "Package_TO_SOT_SMD:SOT-23" H 5050 4525 50  0001 L CIN
-F 3 "https://www.fairchildsemi.com/datasheets/2N/2N7002.pdf" H 4850 4600 50  0001 L CNN
-	1    4850 4600
-	1    0    0    -1
-$EndComp
-Wire Wire Line
-	4950 4800 4950 4850
-Wire Wire Line
-	4950 3950 4950 4050
-Wire Wire Line
-	4950 4350 4950 4400
-Wire Wire Line
-	4250 4050 4250 4000
-Wire Wire Line
-	4250 4050 4450 4050
-$Comp
-L buttonbox2-rescue:DMG3415-custom_comps U?
-U 1 1 5FDBEF04
-P 4150 4150
-AR Path="/5FDBEF04" Ref="U?"  Part="1"
-AR Path="/5FE0503C/5FDBEF04" Ref="U5"  Part="1"
-AR Path="/60BB8BC4/5FDBEF04" Ref="U?"  Part="1"
-F 0 "U5" H 4355 3735 50  0000 L CNN
-F 1 "DMG3415" H 4355 3826 50  0000 L CNN
-F 2 "Package_TO_SOT_SMD:SOT-23" H 4150 4150 50  0001 C CNN
-F 3 "" H 4150 4150 50  0001 C CNN
-	1    4150 4150
-	1    0    0    1
-$EndComp
-Connection ~ 4600 3550
-Wire Wire Line
-	4600 3550 4600 3650
-Wire Wire Line
-	4250 3550 4600 3550
-Wire Wire Line
-	4600 3450 4600 3550
-$Comp
-L power:GND #PWR?
-U 1 1 5FDBEF0F
-P 4950 4850
-AR Path="/5FDBEF0F" Ref="#PWR?"  Part="1"
-AR Path="/5FE0503C/5FDBEF0F" Ref="#PWR017"  Part="1"
-AR Path="/60BB8BC4/5FDBEF0F" Ref="#PWR?"  Part="1"
-F 0 "#PWR017" H 4950 4600 50  0001 C CNN
-F 1 "GND" H 4955 4677 50  0000 C CNN
-F 2 "" H 4950 4850 50  0001 C CNN
-F 3 "" H 4950 4850 50  0001 C CNN
-	1    4950 4850
-	1    0    0    -1
-$EndComp
-Wire Wire Line
-	3950 3800 3900 3800
-Wire Wire Line
-	3900 4600 4650 4600
-Wire Wire Line
-	3900 4600 3850 4600
-Connection ~ 3900 4600
-Connection ~ 4950 4050
-Wire Wire Line
-	3900 3800 3900 4600
+	3400 4200 3350 4200
 $Comp
 L Device:R R?
 U 1 1 5FDBEF1C
-P 3900 4800
+P 3400 4400
 AR Path="/5FDBEF1C" Ref="R?"  Part="1"
 AR Path="/5FE0503C/5FDBEF1C" Ref="R4"  Part="1"
 AR Path="/60BB8BC4/5FDBEF1C" Ref="R?"  Part="1"
-F 0 "R4" H 3970 4846 50  0000 L CNN
-F 1 "10K" H 3970 4755 50  0000 L CNN
-F 2 "Resistor_SMD:R_0805_2012Metric" V 3830 4800 50  0001 C CNN
-F 3 "~" H 3900 4800 50  0001 C CNN
-	1    3900 4800
-	1    0    0    -1
-$EndComp
-Wire Wire Line
-	3900 4650 3900 4600
-Wire Wire Line
-	3900 4950 3900 5000
+F 0 "R4" H 3470 4446 50  0000 L CNN
+F 1 "10K" H 3470 4355 50  0000 L CNN
+F 2 "Resistor_SMD:R_0805_2012Metric" V 3330 4400 50  0001 C CNN
+F 3 "~" H 3400 4400 50  0001 C CNN
+	1    3400 4400
+	1    0    0    -1
+$EndComp
+Wire Wire Line
+	3400 4250 3400 4200
+Wire Wire Line
+	3400 4550 3400 4600
 $Comp
 L power:GND #PWR?
 U 1 1 5FDBEF25
-P 3900 5000
+P 3400 4600
 AR Path="/5FDBEF25" Ref="#PWR?"  Part="1"
 AR Path="/5FE0503C/5FDBEF25" Ref="#PWR015"  Part="1"
 AR Path="/60BB8BC4/5FDBEF25" Ref="#PWR?"  Part="1"
-F 0 "#PWR015" H 3900 4750 50  0001 C CNN
-F 1 "GND" H 3905 4827 50  0000 C CNN
-F 2 "" H 3900 5000 50  0001 C CNN
-F 3 "" H 3900 5000 50  0001 C CNN
-	1    3900 5000
+F 0 "#PWR015" H 3400 4350 50  0001 C CNN
+F 1 "GND" H 3405 4427 50  0000 C CNN
+F 2 "" H 3400 4600 50  0001 C CNN
+F 3 "" H 3400 4600 50  0001 C CNN
+	1    3400 4600
 	1    0    0    -1
 $EndComp
@@
 AR Path="/60BB8BC4/5FE0172D" Ref="R?"  Part="1"
 F 0 "R11" H 8470 3946 50  0000 L CNN
-F 1 "TBD" H 8470 3855 50  0000 L CNN
+F 1 "20K" H 8470 3855 50  0000 L CNN
 F 2 "Resistor_SMD:R_0805_2012Metric" V 8330 3900 50  0001 C CNN
 F 3 "~" H 8400 3900 50  0001 C CNN
@@
 Wire Wire Line
 	8550 4250 8250 4250
-Wire Wire Line
-	4400 4150 4450 4150
-Wire Wire Line
-	4450 4150 4450 4050
-Connection ~ 4450 4050
-Wire Wire Line
-	4450 4050 4950 4050
-Text HLabel 4400 4150 0    50   Input ~ 0
+Text HLabel 4950 4200 3    50   Input ~ 0
 AMP_SHDN
 Text HLabel 8250 4250 0    50   Input ~ 0
@@
 	5600 5250 3350 5250
 Wire Notes Line
-	3350 5250 3350 3150
+	2900 5250 2900 3150
 Text Notes 4250 5200 0    89   ~ 0
 Power
@@
 AR Path="/5FE0503C/5FF0DDDF" Ref="R21"  Part="1"
 AR Path="/60BB8BC4/5FF0DDDF" Ref="R?"  Part="1"
-F 0 "R21" V 7835 2700 50  0000 C CNN
+F 0 "R21" V 8100 2700 50  0000 C CNN
 F 1 "22K" V 7834 2700 50  0001 C CNN
 F 2 "Resistor_SMD:R_0805_2012Metric" V 7880 2700 50  0001 C CNN
@@
 AR Path="/60BB8BC4/618A19C0" Ref="R?"  Part="1"
 F 0 "R2" V 7443 5600 50  0000 C CNN
-F 1 "10K" V 7534 5600 50  0000 C CNN
+F 1 "1K" V 7534 5600 50  0000 C CNN
 F 2 "Resistor_SMD:R_0805_2012Metric" V 7580 5600 50  0001 C CNN
 F 3 "~" H 7650 5600 50  0001 C CNN
@@
 AR Path="/60BB8BC4/618A19EF" Ref="R?"  Part="1"
 F 0 "R3" H 8570 5396 50  0000 L CNN
-F 1 "TBD" H 8570 5305 50  0000 L CNN
+F 1 "20K" H 8570 5305 50  0000 L CNN
 F 2 "Resistor_SMD:R_0805_2012Metric" V 8430 5350 50  0001 C CNN
 F 3 "~" H 8500 5350 50  0001 C CNN
@@
 Text HLabel 7800 2400 2    50   Input ~ 0
 SD_DAT
+Text GLabel 3350 4200 0    50   Input ~ 0
+PLAYER_ON
+$Comp
+L Logic_LevelTranslator:SN74LV1T34DBV U5
+U 1 1 60E5D30C
+P 3900 4200
+F 0 "U5" H 4244 4246 50  0000 L CNN
+F 1 "SN74LV1T34DBV" H 4244 4155 50  0000 L CNN
+F 2 "Package_TO_SOT_SMD:SOT-23-5" H 4550 3950 50  0001 C CNN
+F 3 "https://www.ti.com/lit/ds/symlink/sn74lv1t34.pdf" H 3500 4000 50  0001 C CNN
+	1    3900 4200
+	1    0    0    -1
+$EndComp
+Wire Wire Line
+	4600 3450 4600 3650
+$Comp
+L power:+5V #PWR04
+U 1 1 60E954B9
+P 3900 3900
+AR Path="/5FE0503C/60E954B9" Ref="#PWR04"  Part="1"
+AR Path="/60BB8BC4/60E954B9" Ref="#PWR?"  Part="1"
+F 0 "#PWR04" H 3900 3750 50  0001 C CNN
+F 1 "+5V" H 3915 4073 50  0000 C CNN
+F 2 "" H 3900 3900 50  0001 C CNN
+F 3 "" H 3900 3900 50  0001 C CNN
+	1    3900 3900
+	1    0    0    -1
+$EndComp
+$Comp
+L power:GND #PWR?
+U 1 1 60E959C6
+P 3900 4500
+AR Path="/60E959C6" Ref="#PWR?"  Part="1"
+AR Path="/5FE0503C/60E959C6" Ref="#PWR017"  Part="1"
+AR Path="/60BB8BC4/60E959C6" Ref="#PWR?"  Part="1"
+F 0 "#PWR017" H 3900 4250 50  0001 C CNN
+F 1 "GND" H 3905 4327 50  0000 C CNN
+F 2 "" H 3900 4500 50  0001 C CNN
+F 3 "" H 3900 4500 50  0001 C CNN
+	1    3900 4500
+	1    0    0    -1
+$EndComp
+Wire Wire Line
+	3400 4200 3600 4200
+Connection ~ 3400 4200
+Wire Wire Line
+	4950 4200 4200 4200
+Wire Wire Line
+	4950 3950 4950 4200
 $EndSCHEMATC
