File: buttonbox2.sch (KiCad schematic (older format))
At the start: 29 parts, among them J2 AVR-PDI-6, J4 Conn_01x03_Male, SW1 SW_SP3T, SW3 Rotary_Encoder_Switch, U1 ATxmega256A3-AU, U6 AMS1117-3.3, Y2 Crystal_GND24

Commit message: Added SYS disconnect, routed USB, changed few things
Parts:
- added H1, H2, H3, H4: MountingHole_Pad, MountingHole:MountingHole_2.5mm_Pad, symbol Mechanical:MountingHole_Pad
Connections:
- net GND: now also H1.1, H2.1, H3.1, H4.1
Changed lines of the file:
@@
 STB
 NoConn ~ 3300 3450
+$Comp
+L Mechanical:MountingHole_Pad H4
+U 1 1 60E727AA
+P 5150 4300
+F 0 "H4" H 5250 4349 50  0000 L CNN
+F 1 "MountingHole_Pad" H 5250 4258 50  0000 L CNN
+F 2 "MountingHole:MountingHole_2.5mm_Pad" H 5150 4300 50  0001 C CNN
+F 3 "~" H 5150 4300 50  0001 C CNN
+	1    5150 4300
+	1    0    0    -1
+$EndComp
+$Comp
+L Mechanical:MountingHole_Pad H3
+U 1 1 60E73BB2
+P 4950 4300
+F 0 "H3" H 5050 4349 50  0000 L CNN
+F 1 "MountingHole_Pad" H 5050 4258 50  0000 L CNN
+F 2 "MountingHole:MountingHole_2.5mm_Pad" H 4950 4300 50  0001 C CNN
+F 3 "~" H 4950 4300 50  0001 C CNN
+	1    4950 4300
+	1    0    0    -1
+$EndComp
+$Comp
+L Mechanical:MountingHole_Pad H2
+U 1 1 60E73E82
+P 4750 4300
+F 0 "H2" H 4850 4349 50  0000 L CNN
+F 1 "MountingHole_Pad" H 4850 4258 50  0000 L CNN
+F 2 "MountingHole:MountingHole_2.5mm_Pad" H 4750 4300 50  0001 C CNN
+F 3 "~" H 4750 4300 50  0001 C CNN
+	1    4750 4300
+	1    0    0    -1
+$EndComp
+$Comp
+L Mechanical:MountingHole_Pad H1
+U 1 1 60E7414C
+P 4550 4300
+F 0 "H1" H 4550 4587 50  0000 C CNN
+F 1 "MountingHole_Pad" H 4550 4496 50  0000 C CNN
+F 2 "MountingHole:MountingHole_2.5mm_Pad" H 4550 4300 50  0001 C CNN
+F 3 "~" H 4550 4300 50  0001 C CNN
+	1    4550 4300
+	1    0    0    -1
+$EndComp
+$Comp
+L power:GND #PWR048
+U 1 1 60E74449
+P 4850 4400
+F 0 "#PWR048" H 4850 4150 50  0001 C CNN
+F 1 "GND" H 4855 4227 50  0000 C CNN
+F 2 "" H 4850 4400 50  0001 C CNN
+F 3 "" H 4850 4400 50  0001 C CNN
+	1    4850 4400
+	1    0    0    -1
+$EndComp
+Wire Wire Line
+	4550 4400 4750 4400
+Connection ~ 4750 4400
+Wire Wire Line
+	4750 4400 4850 4400
+Connection ~ 4850 4400
+Wire Wire Line
+	4850 4400 4950 4400
+Connection ~ 4950 4400
+Wire Wire Line
+	4950 4400 5150 4400
 $EndSCHEMATC

Commit message: Changed a lot, ordered the final thing
Parts:
- removed C4: 100n, Capacitor_SMD:C_0805_2012Metric, symbol Device:C
- removed R1: 10K, Resistor_SMD:R_0805_2012Metric, symbol Device:R
- added R1, R41: 220, Resistor_SMD:R_0805_2012Metric, symbol Device:R_Small
- added TP2: TestPoint, TestPoint:TestPoint_THTPad_D2.0mm_Drill1.0mm, symbol Connector:TestPoint
Connections:
- net +3V3: now also TP2.1
- net GND: now also R1.2, R41.2; no longer SW3.C
- net at SW3.S1: now also R41.1; no longer R38.2
- net at C39.1, SW3.S2, U1.13 (PB7): now also R38.2
- net STAT: now reaches U1.17 (PC1)
- net RESET: no longer names the net of J2.5 (CLOCK), U1.57 (~RESET~/PDI_CLK)
- new net: R1.1, SW3.C
- no-connect marks 17 -> 16
Other:
- moved on the sheet: R38
Changed lines of the file:
@@
 Connection ~ 2600 1200
-$Comp
-L power:GND #PWR04
-U 1 1 5FD212C1
-P 8550 3250
-F 0 "#PWR04" H 8550 3000 50  0001 C CNN
-F 1 "GND" H 8555 3077 50  0000 C CNN
-F 2 "" H 8550 3250 50  0001 C CNN
-F 3 "" H 8550 3250 50  0001 C CNN
-	1    8550 3250
-	1    0    0    -1
-$EndComp
 $Comp
 L Device:C C1
@@
 	1    0    0    -1
 $EndComp
-Text GLabel 8600 2850 2    50   Input ~ 0
-RESET
-Wire Wire Line
-	8550 3250 8550 3200
-Wire Wire Line
-	8550 2850 8600 2850
-Connection ~ 8550 2850
-Wire Wire Line
-	8550 2900 8550 2850
-$Comp
-L Device:C C4
-U 1 1 5FD211E3
-P 8550 3050
-F 0 "C4" H 8665 3096 50  0000 L CNN
-F 1 "100n" H 8665 3005 50  0000 L CNN
-F 2 "Capacitor_SMD:C_0805_2012Metric" H 8588 2900 50  0001 C CNN
-F 3 "~" H 8550 3050 50  0001 C CNN
-	1    8550 3050
-	1    0    0    -1
-$EndComp
-Wire Wire Line
-	8550 2800 8550 2850
-Wire Wire Line
-	8550 2450 8550 2500
-$Comp
-L Device:R R1
-U 1 1 5FD1F216
-P 8550 2650
-F 0 "R1" H 8620 2696 50  0000 L CNN
-F 1 "10K" H 8620 2605 50  0000 L CNN
-F 2 "Resistor_SMD:R_0805_2012Metric" V 8480 2650 50  0001 C CNN
-F 3 "~" H 8550 2650 50  0001 C CNN
-	1    8550 2650
-	1    0    0    -1
-$EndComp
 Wire Wire Line
 	1900 1650 1750 1650
@@
 Wire Wire Line
 	1900 1000 1900 1550
-Text GLabel 1900 1200 2    50   Input ~ 0
-RESET
 Text GLabel 1900 3350 0    50   Input ~ 0
 Row1
@@
 $EndComp
 $Comp
-L power:+3.3V #PWR0105
-U 1 1 6180B701
-P 8550 2450
-F 0 "#PWR0105" H 8550 2300 50  0001 C CNN
-F 1 "+3.3V" H 8565 2623 50  0000 C CNN
-F 2 "" H 8550 2450 50  0001 C CNN
-F 3 "" H 8550 2450 50  0001 C CNN
-	1    8550 2450
-	1    0    0    -1
-$EndComp
-$Comp
 L power:+3.3V #PWR0106
 U 1 1 61824272
@@
 L power:GND #PWR055
 U 1 1 60CA3341
-P 4150 2950
-F 0 "#PWR055" H 4150 2700 50  0001 C CNN
-F 1 "GND" H 4155 2777 50  0000 C CNN
-F 2 "" H 4150 2950 50  0001 C CNN
-F 3 "" H 4150 2950 50  0001 C CNN
-	1    4150 2950
-	1    0    0    -1
-$EndComp
-Wire Wire Line
-	4250 2950 4150 2950
+P 4050 3050
+F 0 "#PWR055" H 4050 2800 50  0001 C CNN
+F 1 "GND" H 4055 2877 50  0000 C CNN
+F 2 "" H 4050 3050 50  0001 C CNN
+F 3 "" H 4050 3050 50  0001 C CNN
+	1    4050 3050
+	1    0    0    -1
+$EndComp
+Wire Wire Line
+	4050 2950 4050 3050
 $Comp
 L Device:R R37
@@
 L power:+3V3 #PWR056
 U 1 1 60D421AA
-P 5100 2500
-F 0 "#PWR056" H 5100 2350 50  0001 C CNN
-F 1 "+3V3" H 5115 2673 50  0000 C CNN
-F 2 "" H 5100 2500 50  0001 C CNN
-F 3 "" H 5100 2500 50  0001 C CNN
-	1    5100 2500
-	1    0    0    -1
-$EndComp
-Wire Wire Line
-	4850 2850 5100 2850
-Wire Wire Line
-	5100 2850 5100 2800
+P 5250 2900
+F 0 "#PWR056" H 5250 2750 50  0001 C CNN
+F 1 "+3V3" H 5265 3073 50  0000 C CNN
+F 2 "" H 5250 2900 50  0001 C CNN
+F 3 "" H 5250 2900 50  0001 C CNN
+	1    5250 2900
+	1    0    0    -1
+$EndComp
+Wire Wire Line
+	5250 3250 5250 3200
 Wire Wire Line
 	4900 3050 4900 3250
@@
 L Device:R R38
 U 1 1 60D8FC06
-P 5100 2650
-F 0 "R38" H 5170 2696 50  0000 L CNN
-F 1 "10K" H 5170 2605 50  0000 L CNN
-F 2 "Resistor_SMD:R_0805_2012Metric" V 5030 2650 50  0001 C CNN
-F 3 "~" H 5100 2650 50  0001 C CNN
-	1    5100 2650
+P 5250 3050
+F 0 "R38" H 5320 3096 50  0000 L CNN
+F 1 "10K" H 5320 3005 50  0000 L CNN
+F 2 "Resistor_SMD:R_0805_2012Metric" V 5180 3050 50  0001 C CNN
+F 3 "~" H 5250 3050 50  0001 C CNN
+	1    5250 3050
 	1    0    0    -1
 $EndComp
@@
 Text GLabel 3300 3750 2    50   Input ~ 0
 STB
-NoConn ~ 3300 3450
 $Comp
 L Mechanical:MountingHole_Pad H4
@@
 Wire Wire Line
 	4950 4400 5150 4400
+Wire Wire Line
+	4900 3250 5250 3250
+Connection ~ 4900 3250
+$Comp
+L power:GND #PWR0105
+U 1 1 60D1BDC8
+P 5050 3100
+F 0 "#PWR0105" H 5050 2850 50  0001 C CNN
+F 1 "GND" H 5055 2927 50  0000 C CNN
+F 2 "" H 5050 3100 50  0001 C CNN
+F 3 "" H 5050 3100 50  0001 C CNN
+	1    5050 3100
+	1    0    0    -1
+$EndComp
+$Comp
+L Device:R_Small R41
+U 1 1 60D2E125
+P 5050 3000
+F 0 "R41" H 5109 3046 50  0000 L CNN
+F 1 "220" H 5109 2955 50  0000 L CNN
+F 2 "Resistor_SMD:R_0805_2012Metric" H 5050 3000 50  0001 C CNN
+F 3 "~" H 5050 3000 50  0001 C CNN
+	1    5050 3000
+	1    0    0    -1
+$EndComp
+Wire Wire Line
+	4850 2850 5050 2850
+Wire Wire Line
+	5050 2850 5050 2900
+$Comp
+L Device:R_Small R1
+U 1 1 60D3D6B8
+P 4150 2950
+F 0 "R1" V 3954 2950 50  0000 C CNN
+F 1 "220" V 4045 2950 50  0000 C CNN
+F 2 "Resistor_SMD:R_0805_2012Metric" H 4150 2950 50  0001 C CNN
+F 3 "~" H 4150 2950 50  0001 C CNN
+	1    4150 2950
+	0    1    1    0
+$EndComp
+$Comp
+L Connector:TestPoint TP?
+U 1 1 60E044AD
+P 8200 2750
+AR Path="/60E90241/60E044AD" Ref="TP?"  Part="1"
+AR Path="/60E044AD" Ref="TP2"  Part="1"
+F 0 "TP2" H 8142 2776 50  0000 R CNN
+F 1 "TestPoint" H 8142 2867 50  0000 R CNN
+F 2 "TestPoint:TestPoint_THTPad_D2.0mm_Drill1.0mm" H 8400 2750 50  0001 C CNN
+F 3 "~" H 8400 2750 50  0001 C CNN
+	1    8200 2750
+	-1   0    0    1
+$EndComp
+Connection ~ 8200 2750
+Text GLabel 3300 3450 2    50   Input ~ 0
+STAT
 $EndSCHEMATC

Commit message: Added SchroombortFirmware folder
Parts:
- Cams1: value C -> 1uF
Changed lines of the file:
@@
 P 7250 2900
 F 0 "Cams1" H 7365 2946 50  0000 L CNN
-F 1 "C" H 7365 2855 50  0000 L CNN
+F 1 "1uF" H 7365 2855 50  0000 L CNN
 F 2 "Capacitor_SMD:C_0805_2012Metric" H 7288 2750 50  0001 C CNN
 F 3 "~" H 7250 2900 50  0001 C CNN
